File: schematic/rpm_generator.kicad_sch (KiCad schematic)
At the start: 1 part

Commit message: Update schematic
Connections:
- net neg renamed b
- net pos renamed a
Changed lines of the file:
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@@
 (kicad_sch
-	(version 20231120)
+	(version 20250114)
 	(generator "eeschema")
-	(generator_version "8.0")
+	(generator_version "9.0")
 	(paper "A4")
 	(title_block
@@
 		(rev "1.0")
 		(company "Michael Büsch <m@bues.ch>")
+	)
+	(text "4-pole rotating magnet\ninduces current into L"
+		(exclude_from_sim no)
+		(at 144.526 68.326 0)
+		(effects
+			(font
+				(size 1.27 1.27)
+			)
+		)
 	)
 	(wire
@@
 		)
 	)
-	(text "4-pole rotating magnet\ninduces current into L"
-		(exclude_from_sim no)
-		(at 144.526 68.326 0)
-		(effects
-			(font
-				(size 1.27 1.27)
-			)
-		)
-	)
-	(hierarchical_label "neg"
+	(hierarchical_label "b"
 		(shape input)
 		(at 152.4 90.17 270)
-		(fields_autoplaced yes)
 		(effects
 			(font
@@
 		)
 	)
-	(hierarchical_label "pos"
+	(hierarchical_label "a"
 		(shape input)
 		(at 137.16 90.17 270)
-		(fields_autoplaced yes)
 		(effects
 			(font
