File: schematic/ntc.kicad_sch (KiCad schematic)
At the start: 2 parts

Commit message: schematic: Assign some footprints
Parts:
- R17: footprint (none) -> Resistor_THT:R_Axial_DIN0207_L6.3mm_D2.5mm_P2.54mm_Vertical
Changed lines of the file:
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@@
 			)
 		)
-		(property "Footprint" ""
+		(property "Footprint" "Resistor_THT:R_Axial_DIN0207_L6.3mm_D2.5mm_P2.54mm_Vertical"
 			(at 130.81 123.952 90)
 			(hide yes)
